Commit message: Add automatic homing from rest position and Viser visualization

File: factr_interface/urdf/factr_teleop_franka.urdf (robot description, URDF)
Before this commit: robot factr_teleop_franka, 8 links, 7 joints
Joints:
- joint joint_2: limit lower=-1.7628 upper=1.7628 effort=0.92 velocity=6.8 -> lower=-1.52 upper=1.7628 effort=0.92 velocity=6.8
- joint joint_4: limit lower=-3.0718 upper=-0.0698 effort=0.92 velocity=6.8 -> lower=-3.14 upper=-0.0698 effort=0.92 velocity=6.8
