Commit message: Consolidate inheritance from base Factr class

File: urdf/factr_teleop_franka.urdf (robot description, URDF)
Before this commit: robot factr_teleop_franka, 8 links, 7 joints
Links:
- link base_link: geometry collision mesh filename=package://factr_interface/urdf/meshes/base_link.STL; visual mesh filename=package://factr_interface/urdf/meshes/base_link.STL
- link link_1: geometry collision mesh filename=package://factr_interface/urdf/meshes/link_1.STL; visual mesh filename=package://factr_interface/urdf/meshes/link_1.STL
- link link_2: geometry collision mesh filename=package://factr_interface/urdf/meshes/link_2.STL; visual mesh filename=package://factr_interface/urdf/meshes/link_2.STL
- link link_3: geometry collision mesh filename=package://factr_interface/urdf/meshes/link_3.STL; visual mesh filename=package://factr_interface/urdf/meshes/link_3.STL
- link link_4: geometry collision mesh filename=package://factr_interface/urdf/meshes/link_4.STL; visual mesh filename=package://factr_interface/urdf/meshes/link_4.STL
- link link_5: geometry collision mesh filename=package://factr_interface/urdf/meshes/link_5.STL; visual mesh filename=package://factr_interface/urdf/meshes/link_5.STL
- link link_6: geometry collision mesh filename=package://factr_interface/urdf/meshes/link_6.STL; visual mesh filename=package://factr_interface/urdf/meshes/link_6.STL
- link link_7: geometry collision mesh filename=package://factr_interface/urdf/meshes/link_7.STL; visual mesh filename=package://factr_interface/urdf/meshes/link_7.STL
